Commit message: fix yaml file, fix joint state publisher, and added movement to turtle robot

File: src/install/turtle_brick/share/turtle_brick/turtle.urdf.xacro (robot description, xacro)
@@ -121,5 +121,5 @@
         <parent link="stem"/>
         <child link="wheel"/>
-        <origin xyz="0 0 -0.7" rpy="0 0 0"/>
+        <origin xyz="0 0 ${-(wradius+width/2+stem_length)}" rpy="0 0 0"/>
     </joint>
 </robot>
