Commit message: added the unreachable mark and fixed some boundary bugs

File: install/turtle_brick/share/turtle_brick/turtle.urdf.xacro (robot description, xacro)
@@ -56,14 +56,14 @@
     <link name="fix_link">
         <visual>
-        <origin xyz="0 0 ${width/2+(platform_h-wradius-stem_length-width-length)/2}" rpy="0 0 0" />
+        <origin xyz="0 0 ${width/2+(platform_h-wradius*2-stem_length-width-length)/2}" rpy="0 0 0" />
         <geometry>
-            <cylinder radius="${sradius}" length="${platform_h-wradius-stem_length-width-length}" />
+            <cylinder radius="${sradius}" length="${platform_h-wradius*2-stem_length-width-length}" />
         </geometry>
         <material name="red"/>
         </visual>
         <collision>
-            <origin xyz="0 0 ${width/2+(platform_h-wradius-stem_length-width-length)/2}" rpy="0 0 0"/>
+            <origin xyz="0 0 ${width/2+(platform_h-wradius*2-stem_length-width-length)/2}" rpy="0 0 0"/>
             <geometry>
-                <cylinder radius="${sradius}" length="${platform_h-wradius-stem_length-width-length}" />
+                <cylinder radius="${sradius}" length="${platform_h-wradius*2-stem_length-width-length}" />
             </geometry>
         </collision>
@@ -105,5 +105,5 @@
     </joint>
     <joint name='link_platform1' type="continuous">
-        <origin xyz="0 0 ${width/2+(platform_h-wradius-stem_length-width-length/2)}" rpy="0 0 0"/>
+        <origin xyz="0 0 ${width/2+(platform_h-wradius*2-stem_length-width-length/2)}" rpy="0 0 0"/>
         <parent link="fix_link"/>
         <child link="platform"/>

Commit message: stem and wheel turn and added to readme

File: install/turtle_brick/share/turtle_brick/turtle.urdf.xacro (robot description, xacro)
@@ -22,5 +22,5 @@
     </material>
     <material name="black">
-        <color rgba="0.0 0.0 0.0 1.0"/>
+        <color rgba="0.2 0.2 0.2 1.0"/>
     </material>
     <link name="base_link">
@@ -86,5 +86,5 @@
     <link name="wheel">
         <visual>
-            <origin xyz="0 0 0" rpy="0 ${pi/2} 0" />
+            <origin xyz="0 0 0" rpy="${pi/2}  0 0" />
             <geometry>
                 <cylinder radius="${wradius}" length="0.1" />
@@ -93,5 +93,5 @@
         </visual>
         <collision>
-            <origin xyz="0 0 0" rpy="0 ${pi/2} 0"/>
+            <origin xyz="0 0 0" rpy="${pi/2} 0 0"/>
             <geometry>
                 <cylinder radius="${wradius}" length="0.1" />
@@ -117,5 +117,5 @@
     </joint>
     <joint name='stem_wheel' type="continuous">
-        <axis xyz="1 0 0"/>
+        <axis xyz="0 1 0"/>
         <limit effort="1000.0" velocity="${max_vel/wradius}"/>
         <parent link="stem"/>

Commit message: fixed style errors

File: install/turtle_brick/share/turtle_brick/turtle.urdf.xacro (robot description, xacro)
@@ -3,5 +3,5 @@
     <xacro:property name="yaml_file" value="$(find turtle_brick)/config/turtle.yaml" />
     <xacro:property name="turtle" value="${load_yaml(yaml_file)}" />
-    <xacro:property name="platform_h"  value="${turtle['/**']['ros__parameters']['platform_height']}" /> <!-- ${turtle['platform_height']} 1.7 -->
+    <xacro:property name="platform_h"  value="${turtle['/**']['ros__parameters']['platform_height']}" />
     <xacro:property name="width" value="0.5"/>
     <xacro:property name="length" value="0.1"/>
@@ -9,7 +9,7 @@
     <xacro:property name="pradius" value="0.35"/>
     <xacro:property name="sradius" value="0.1"/>
-    <xacro:property name="wradius" value="${turtle['/**']['ros__parameters']['wheel_radius']}"/> <!-- ${turtle['wheel_radius']} 0.3 -->
+    <xacro:property name="wradius" value="${turtle['/**']['ros__parameters']['wheel_radius']}"/>
     <xacro:property name="force" value="100.0"/>
-    <xacro:property name="max_vel" value="${turtle['/**']['ros__parameters']['max_velocity']}"/>  <!--${turtle['max_velocity']} 0.22-->
+    <xacro:property name="max_vel" value="${turtle['/**']['ros__parameters']['max_velocity']}"/>
     <material name="blue">
         <color rgba="0 0 1.0 1.0"/>

File: src/install/turtle_brick/share/turtle_brick/turtle.urdf.xacro (robot description, xacro)
@@ -22,5 +22,5 @@
     </material>
     <material name="black">
-        <color rgba="0.0 0.0 0.0 1.0"/>
+        <color rgba="0.2 0.2 0.2 1.0"/>
     </material>
     <link name="base_link">
@@ -56,14 +56,14 @@
     <link name="fix_link">
         <visual>
-        <origin xyz="0 0 ${width/2+(platform_h-wradius-stem_length-width-length)/2}" rpy="0 0 0" />
+        <origin xyz="0 0 ${width/2+(platform_h-wradius*2-stem_length-width-length)/2}" rpy="0 0 0" />
         <geometry>
-            <cylinder radius="${sradius}" length="${platform_h-wradius-stem_length-width-length}" />
+            <cylinder radius="${sradius}" length="${platform_h-wradius*2-stem_length-width-length}" />
         </geometry>
         <material name="red"/>
         </visual>
         <collision>
-            <origin xyz="0 0 ${width/2+(platform_h-wradius-stem_length-width-length)/2}" rpy="0 0 0"/>
+            <origin xyz="0 0 ${width/2+(platform_h-wradius*2-stem_length-width-length)/2}" rpy="0 0 0"/>
             <geometry>
-                <cylinder radius="${sradius}" length="${platform_h-wradius-stem_length-width-length}" />
+                <cylinder radius="${sradius}" length="${platform_h-wradius*2-stem_length-width-length}" />
             </geometry>
         </collision>
@@ -86,5 +86,5 @@
     <link name="wheel">
         <visual>
-            <origin xyz="0 0 0" rpy="0 ${pi/2} 0" />
+            <origin xyz="0 0 0" rpy="${pi/2}  0 0" />
             <geometry>
                 <cylinder radius="${wradius}" length="0.1" />
@@ -93,5 +93,5 @@
         </visual>
         <collision>
-            <origin xyz="0 0 0" rpy="0 ${pi/2} 0"/>
+            <origin xyz="0 0 0" rpy="${pi/2} 0 0"/>
             <geometry>
                 <cylinder radius="${wradius}" length="0.1" />
@@ -105,5 +105,5 @@
     </joint>
     <joint name='link_platform1' type="continuous">
-        <origin xyz="0 0 ${width/2+(platform_h-wradius-stem_length-width-length/2)}" rpy="0 0 0"/>
+        <origin xyz="0 0 ${width/2+(platform_h-wradius*2-stem_length-width-length/2)}" rpy="0 0 0"/>
         <parent link="fix_link"/>
         <child link="platform"/>
@@ -117,5 +117,5 @@
     </joint>
     <joint name='stem_wheel' type="continuous">
-        <axis xyz="1 0 0"/>
+        <axis xyz="0 1 0"/>
         <limit effort="1000.0" velocity="${max_vel/wradius}"/>
         <parent link="stem"/>
